File: ESP32-ANalog/ESP32-ANalog.kicad_sch (KiCad schematic)
At the start: 0 parts

Commit message: Refactor code structure for improved readability and maintainability
Parts:
- added BZ1: Buzzer, symbol Device:Buzzer
- added C1: 1nF, Capacitor_SMD:C_0603_1608Metric, symbol Device:C_Small
- added LDR1: LDR07, OptoDevice:R_LDR_5.1x4.3mm_P3.4mm_Vertical, symbol Sensor_Optical:LDR07
- added Q1: 2N3904, Package_TO_SOT_THT:TO-92_Inline, symbol Transistor_BJT:2N3904
- added R1: 10k Ohm, symbol Device:R_Small_US
- added R2: 470 Ohm, symbol Device:R_Small_US
- added U1: ESP32-WROOM-32, RF_Module:ESP32-WROOM-32, symbol RF_Module:ESP32-WROOM-32
Connections:
- new net: BZ1.2 (-), Q1.3 (C)
- new net: Q1.2 (B), R1.2
- new net: R1.1, U1.30 (IO18)
- new net: U1.1 (GND), U1.15 (GND), U1.38 (GND), U1.39 (GND)
- new net: C1.1, LDR1.2, R2.2, U1.7 (IO35)
- new net +3.3V: BZ1.1 (+), LDR1.1
- new net GND: C1.2, Q1.1 (E), R2.1
Other:
- note added: "LDR (10 mm)"
- note added: "R = 100 ~ 500k OHM @100 OHM -> Vout = 3.26V @500k OHM -> Vout = 0.06V"
